File: kim-1-mtu-motherboard/kim-1-mtu-motherboard.kicad_sch (KiCad schematic)
At the start: 105 parts, among them J1 Audio Loop, J1 Power_Connector, J10 GND, J11 K7, J12 DECEN, J13 K7, J14 DECEN, J2 Audio HI/LO, J4 Audio Out, J5 Audio In, J7 Daughterboard, J7 Decode, J8 RESET, J9 GND, P1 EXP_BOARD, P1 KIM_EXP, P10 EXP_BOARD, P11 EXP_BOARD, P12 KIM-1, P14 KIM_APPL, P2 EXP_BOARD, P3 EXP_BOARD, P4 EXP_BOARD, P5 EXP_BOARD, P6 KIM-1, P7 EXP_BOARD, P8 EXP_BOARD, P9 EXP_BOARD, U1 74HCT541, U2 74HCT541, U3 74HCT541, U4 74LS245, U5 74LS07

Commit message: Disable data bus transceiver when DECEN or K7 active (low). Should fix issue #2
Parts:
- added C64: 100nF, Capacitor_THT:C_Disc_D5.0mm_W2.5mm_P5.00mm, symbol Device:C_Small
- added U6: 74LS00, Package_DIP:DIP-14_W7.62mm_LongPads, symbol 74xx:74LS00
Connections:
- net +5V: now also C64.1, U6.14 (VCC)
- net DECEN: now also U6.10
- net GND: now also C64.2, U6.1, U6.12, U6.13, U6.2, U6.4, U6.5, U6.7 (GND); no longer U4.19 (CE)
- net K7: now also U6.9
- new net: U4.19 (CE), U6.8
- no-connect marks 18 -> 21
Other:
- moved on the sheet: C1, C2, C3, C4, C5, J1, J10, J2, J4, J5, J7, J9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
