File: kim-1-aux-card-usb/kim-1-aux-card-usb.kicad_sch (KiCad schematic)
At the start: 30 parts, among them J1 Motherboard, J11 USB_C_Receptacle_USB2.0, J2 SD_Shield, J4 Reset, J5 GND, J6 +5V, J6 DIN-6, J8 USB_TTL, J9 TTL_SERIAL, Q1 PN2222A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

Commit message: Revision 3. Fixes Issue #3
Parts:
- added SW2: SD_IEC, Button_Switch_THT:SW_DIP_SPSTx02_Slide_9.78x7.26mm_W7.62mm_P2.54mm, symbol Switch:SW_DIP_x02
Connections:
- net PA6: now also SW2.2; no longer J6.4, RN1.7 (R6.2), U1.4
- net PA7: now also SW2.1; no longer J6.5, RN1.6 (R5.2), U1.6
- new net: J6.4, RN1.7 (R6.2), SW2.3, U1.4
- new net: J6.5, RN1.6 (R5.2), SW2.4, U1.6
Changed lines of the file:
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@@
     (stroke (width 0) (type default))
   )
-  (bus_entry (at 43.18 181.61) (size 2.54 2.54)
+  (bus_entry (at 43.18 184.785) (size 2.54 2.54)
     (stroke (width 0) (type default))
   )
@@
     (stroke (width 0) (type default))
   )
-  (wire (pts (xy 45.72 184.15) (xy 99.06 184.15))
+  (wire (pts (xy 45.72 187.325) (xy 54.61 187.325))
     (stroke (width 0) (type default))
   )
@@
     (stroke (width 0) (type default))
   )
-  (bus (pts (xy 43.18 181.61) (xy 43.18 187.325))
+  (bus (pts (xy 43.18 184.785) (xy 43.18 187.325))
     (stroke (width 0) (type default))
   )
@@
     (stroke (width 0) (type default))
   )
-  (bus (pts (xy 43.18 175.26) (xy 43.18 181.61))
+  (bus (pts (xy 43.18 175.26) (xy 43.18 184.785))
     (stroke (width 0) (type default))
   )
@@
     (stroke (width 0) (type default))
   )
+  (wire (pts (xy 69.85 189.865) (xy 115.57 189.865))
+    (stroke (width 0) (type default))
+  )
   (wire (pts (xy 34.29 34.925) (xy 40.64 34.925))
     (stroke (width 0) (type default))
@@
     (stroke (width 0) (type default))
   )
+  (wire (pts (xy 69.85 187.325) (xy 99.06 187.325))
+    (stroke (width 0) (type default))
+  )
   (bus (pts (xy 43.18 187.325) (xy 43.18 188.595))
     (stroke (width 0) (type default))
@@
     (stroke (width 0) (type default))
   )
-  (wire (pts (xy 45.72 189.865) (xy 115.57 189.865))
+  (wire (pts (xy 45.72 189.865) (xy 54.61 189.865))
     (stroke (width 0) (type default))
   )
@@
     (stroke (width 0) (type default))
   )
-  (wire (pts (xy 99.06 184.15) (xy 99.06 172.72))
+  (wire (pts (xy 99.06 187.325) (xy 99.06 172.72))
     (stroke (width 0) (type default))
   )
@@
     (effects (font (size 1 1)) (justify left bottom))
   )
-  (label "PA6" (at 45.72 184.15 0) (fields_autoplaced)
+  (label "PA6" (at 45.72 187.325 0) (fields_autoplaced)
     (effects (font (size 1 1)) (justify left bottom))
   )
@@
         )
       )
+    )
+  )
+  (symbol (lib_id "Switch:SW_DIP_x02") (at 62.23 187.325 0) (mirror x) (unit 1)
+    (in_bom yes) (on_board yes) (dnp no)
+    (property "Reference" "SW2" (at 62.23 196.85 0)
+      (effects (font (size 1.27 1.27)))
+    )
+    (property "Value" "SD_IEC" (at 62.23 194.31 0)
+      (effects (font (size 1.27 1.27)))
+    )
+    (property "Footprint" "Button_Switch_THT:SW_DIP_SPSTx02_Slide_9.78x7.26mm_W7.62mm_P2.54mm" (at 62.23 187.325 0)
+      (effects (font (size 1.27 1.27)) hide)
+    )
+    (property "Datasheet" "~" (at 62.23 187.325 0)
+      (effects (font (size 1.27 1.27)) hide)
+    )
+    (pin "1")
+    (pin "2")
+    (pin "3")
+    (pin "4")
+    (instances
+      (project "kim-1-aux-card-usb"
+        (path "/bccd745c-1975-422e-9da9-e7805ccc3aa8"
+          (reference "SW2") (unit 1)
+        )
+      )
